File: tpkbd.kicad_pcb (KiCad board)
At the start: 2 copper layers, 19 parts, among them CON1 AVR-ISP-6, J1 CONN_01X02, J2 CONN_01X01, J3 USB_OTG, J4 CONN_02X20, J5 CONN_01X04, U1 ATMEGA8515-16AU, U2 AP111733, Y1 Crystal_GND24

Commit message: seems complete :)
Parts:
- added J6: GS2, Capacitors_SMD:C_0402, F.Cu at (85.9, 41.1)
- added J7: 0, Capacitors_SMD:C_0402, F.Cu at (56.2, 29.5)
- moved C2 56.5 mm to (79.4, 61.0)
- moved R5 56.5 mm to (86.8, 45.0), turned to 60 degrees
- moved C1 51.7 mm to (68.2, 59.8), turned to 90 degrees
- moved J5 46.4 mm to (61.0, 50.2)
- moved C5 35.6 mm to (64.8, 44.4), turned to 270 degrees
- moved C4 34.8 mm to (65.8, 39.6), turned to 45 degrees
- moved Y1 34.7 mm to (72.8, 60.0)
- moved R1 33.2 mm to (60.8, 46.8)
- moved R4 31.3 mm to (63.2, 35.4), turned to 90 degrees
- moved U2 29.5 mm to (58.4, 42.0), turned to 90 degrees
- moved R3 28.7 mm to (60.6, 35.4), turned to 270 degrees
- moved R2 26.6 mm to (58.4, 35.4), turned to 270 degrees
- moved CON1 25.6 mm to (55.9, 50.2)
- moved J2 23.5 mm to (55.8, 32.6)
- moved J1 21.2 mm to (65.0, 53.6), turned to 90 degrees
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Connections:
- net Net-(J5-Pad3) renamed /tp_rst_b
- J3 pad 5: GND -> Net-(J3-Pad5)
- U1 pad 10: /tp_data -> /kb_id0
- U1 pad 11: /tp_ck -> /kb_id1
- U1 pad 27: /kb_id1 -> /tp_data
- U1 pad 29: /kb_id0 -> /tp_ck
- U1 pad 39: GND -> (no net)
Routing:
- net GND: track 14.9 -> 162.3 mm, vias 0 -> 1
- net +3V3: track 2.79 -> 108.5 mm, vias 0 -> 3
- net +5V: track 0.00 -> 79.9 mm, vias 0 -> 2
- net /C0: track 0.00 -> 75.2 mm
- net /C1: track 0.00 -> 71.0 mm
- net /C2: track 0.00 -> 67.1 mm
- net /C3: track 0.00 -> 63.0 mm
- net /C4: track 0.00 -> 58.7 mm
- net /tp_rst_b: track 0.00 -> 56.6 mm, vias 0 -> 2
- net /hotkey: track 0.00 -> 52.7 mm, vias 0 -> 2
- net /C5: track 0.00 -> 51.8 mm
- net Net-(R3-Pad2): track 0.00 -> 51.2 mm
- net /power: track 0.00 -> 50.2 mm, vias 0 -> 2
- net /C6: track 0.00 -> 48.6 mm
- net /C7: track 0.00 -> 45.5 mm
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- added copper zone on B.Cu, net GND
- added copper zone on F.Cu, net GND
Other:
- board outline added: 43 x 38 mm
- net class Default: clearance 0.3 -> 0.235; via_dia 0.6 -> 1
- net class narrow added: clearance 0.2, trace_width 0.3, via_dia 1, via_drill 0.4
- net class power: via_dia 0.6 -> 1
- net class power-narrow added: clearance 0.2, trace_width 0.4, via_dia 1, via_drill 0.4
- rule trace_clearance: 0.3 -> 0.235
